File: CH552-USB-Devboard/CH552-USB-Devboard.sch (KiCad schematic (older format))
At the start: 45 parts, among them J1 Conn_01x11_Male, J2 Conn_01x11_Male, J3 USB_C_Receptacle, J4 USB_C_Receptacle, SW1 SW_Push, SW2 SW_Push, U1 CH552T, U2 CH552G

Commit message: update PCB
Parts:
- C5, C6: renamed from C?; footprint Capacitor_SMD:C_1206_3216Metric_Pad1.33x1.80mm_HandSolder -> Capacitor_SMD:C_1206_3216Metric_Pad1.42x1.75mm_HandSolder
- R11, R13, R14: renamed from R?; footprint Resistor_SMD:R_0603_1608Metric_Pad0.98x0.95mm_HandSolder -> Resistor_SMD:R_0603_1608Metric_Pad1.05x0.95mm_HandSolder
- gave numbers to parts that had none: 4
Changed lines of the file:
@@
 EESchema Schematic File Version 4
-EELAYER 30 0
+LIBS:CH552-USB-Devboard-cache
+EELAYER 29 0
 EELAYER END
 $Descr A4 11693 8268
@@
 	2400 4100 2500 4100
 $Comp
-L CH552-USB-Devboard:TPS7A4101DGNT U?
+L CH552-USB-Devboard:TPS7A4101DGNT U3
 U 1 1 60D4C1D8
 P 8150 950
-F 0 "U?" H 8150 1315 50  0000 C CNN
+F 0 "U3" H 8150 1315 50  0000 C CNN
 F 1 "TPS7A4101DGNT" H 8150 1224 50  0000 C CNN
 F 2 "CH552-USB-Devboard:HVSSOP-8_3.0x3.0mm_P0.65mm" H 8150 950 50  0001 C CNN
@@
 $EndComp
 $Comp
-L power:GND #PWR?
+L power:GND #PWR0132
 U 1 1 60D4FB76
 P 8050 1250
-F 0 "#PWR?" H 8050 1000 50  0001 C CNN
+F 0 "#PWR0132" H 8050 1000 50  0001 C CNN
 F 1 "GND" H 8055 1077 50  0000 C CNN
 F 2 "" H 8050 1250 50  0001 C CNN
@@
 $EndComp
 $Comp
-L power:GND #PWR?
+L power:GND #PWR0133
 U 1 1 60D52375
 P 8250 1250
-F 0 "#PWR?" H 8250 1000 50  0001 C CNN
+F 0 "#PWR0133" H 8250 1000 50  0001 C CNN
 F 1 "GND" H 8255 1077 50  0000 C CNN
 F 2 "" H 8250 1250 50  0001 C CNN
@@
 $EndComp
 $Comp
-L power:VBUS #PWR?
+L power:VBUS #PWR0134
 U 1 1 60D52A16
 P 7750 1050
-F 0 "#PWR?" H 7750 900 50  0001 C CNN
+F 0 "#PWR0134" H 7750 900 50  0001 C CNN
 F 1 "VBUS" H 7765 1223 50  0000 C CNN
 F 2 "" H 7750 1050 50  0001 C CNN
@@
 $EndComp
 $Comp
-L power:VBUS #PWR?
+L power:VBUS #PWR0135
 U 1 1 60D53623
 P 7450 750
-F 0 "#PWR?" H 7450 600 50  0001 C CNN
+F 0 "#PWR0135" H 7450 600 50  0001 C CNN
 F 1 "VBUS" H 7465 923 50  0000 C CNN
 F 2 "" H 7450 750 50  0001 C CNN
@@
 	7450 850  7450 750
 $Comp
-L power:GND #PWR?
+L power:GND #PWR0136
 U 1 1 60D5DBAE
 P 7450 1300
-F 0 "#PWR?" H 7450 1050 50  0001 C CNN
+F 0 "#PWR0136" H 7450 1050 50  0001 C CNN
 F 1 "GND" H 7455 1127 50  0000 C CNN
 F 2 "" H 7450 1300 50  0001 C CNN
@@
 $EndComp
 $Comp
-L Device:C_Small C?
+L Device:C_Small C5
 U 1 1 60D5E392
 P 7450 1000
-F 0 "C?" H 7542 1046 50  0000 L CNN
+F 0 "C5" H 7542 1046 50  0000 L CNN
 F 1 "4u7, 50V" H 7542 955 50  0000 L CNN
-F 2 "Capacitor_SMD:C_1206_3216Metric_Pad1.33x1.80mm_HandSolder" H 7450 1000 50  0001 C CNN
+F 2 "Capacitor_SMD:C_1206_3216Metric_Pad1.42x1.75mm_HandSolder" H 7450 1000 50  0001 C CNN
 F 3 "~" H 7450 1000 50  0001 C CNN
 F 4 "C29823" H 7450 1000 50  0001 C CNN "LCSC"
@@
 Connection ~ 7450 850
 $Comp
-L Device:C_Small C?
+L Device:C_Small C6
 U 1 1 60D785AE
 P 7450 1200
-F 0 "C?" H 7542 1246 50  0000 L CNN
+F 0 "C6" H 7542 1246 50  0000 L CNN
 F 1 "4u7, 50V" H 7542 1155 50  0000 L CNN
-F 2 "Capacitor_SMD:C_1206_3216Metric_Pad1.33x1.80mm_HandSolder" H 7450 1200 50  0001 C CNN
+F 2 "Capacitor_SMD:C_1206_3216Metric_Pad1.42x1.75mm_HandSolder" H 7450 1200 50  0001 C CNN
 F 3 "~" H 7450 1200 50  0001 C CNN
 F 4 "C29823" H 7450 1200 50  0001 C CNN "LCSC"
@@
 $EndComp
 $Comp
-L Device:C_Small C?
+L Device:C_Small C10
 U 1 1 60D7B491
 P 9400 950
-F 0 "C?" H 9492 996 50  0000 L CNN
+F 0 "C10" H 9492 996 50  0000 L CNN
 F 1 "10uF" H 9492 905 50  0000 L CNN
 F 2 "Capacitor_SMD:C_0603_1608Metric_Pad1.05x0.95mm_HandSolder" H 9400 950 50  0001 C CNN
@@
 $EndComp
 $Comp
-L Device:C_Small C?
+L Device:C_Small C9
 U 1 1 60D813D2
 P 9000 950
-F 0 "C?" H 9092 996 50  0000 L CNN
+F 0 "C9" H 9092 996 50  0000 L CNN
 F 1 "100nF" H 9092 905 50  0000 L CNN
 F 2 "Capacitor_SMD:C_0603_1608Metric_Pad1.05x0.95mm_HandSolder" H 9000 950 50  0001 C CNN
@@
 $EndComp
 $Comp
-L Device:C_Small C?
+L Device:C_Small C8
 U 1 1 60D9BB03
 P 8650 950
-F 0 "C?" H 8742 996 50  0000 L CNN
+F 0 "C8" H 8742 996 50  0000 L CNN
 F 1 "10nF" H 8742 905 50  0000 L CNN
 F 2 "Capacitor_SMD:C_0603_1608Metric_Pad1.05x0.95mm_HandSolder" H 8650 950 50  0001 C CNN
@@
 	9400 850  9400 750
 $Comp
-L power:VCC #PWR?
+L power:VCC #PWR0137
 U 1 1 60DE56D5
 P 9400 750
-F 0 "#PWR?" H 9400 600 50  0001 C CNN
+F 0 "#PWR0137" H 9400 600 50  0001 C CNN
 F 1 "VCC" H 9417 923 50  0000 C CNN
 F 2 "" H 9400 750 50  0001 C CNN
@@
 $EndComp
 $Comp
-L power:GND #PWR?
+L power:GND #PWR0138
 U 1 1 60DE7792
 P 9000 1050
-F 0 "#PWR?" H 9000 800 50  0001 C CNN
+F 0 "#PWR0138" H 9000 800 50  0001 C CNN
 F 1 "GND" H 9005 877 50  0000 C CNN
 F 2 "" H 9000 1050 50  0001 C CNN
@@
 $EndComp
 $Comp
-L power:GND #PWR?
+L power:GND #PWR0139
 U 1 1 60DE7DCD
 P 9400 1050
-F 0 "#PWR?" H 9400 800 50  0001 C CNN
+F 0 "#PWR0139" H 9400 800 50  0001 C CNN
 F 1 "GND" H 9405 877 50  0000 C CNN
 F 2 "" H 9400 1050 50  0001 C CNN
@@
 $EndComp
 $Comp
-L Device:R_Small R?
+L Device:R_Small R11
 U 1 1 60DE8346
 P 9750 950
-F 0 "R?" V 9554 950 50  0000 C CNN
+F 0 "R11" V 9554 950 50  0000 C CNN
 F 1 "62k" V 9645 950 50  0000 C CNN
-F 2 "Resistor_SMD:R_0603_1608Metric_Pad0.98x0.95mm_HandSolder" H 9750 950 50  0001 C CNN
+F 2 "Resistor_SMD:R_0603_1608Metric_Pad1.05x0.95mm_HandSolder" H 9750 950 50  0001 C CNN
 F 3 "~" H 9750 950 50  0001 C CNN
 F 4 "C23221" V 9750 950 50  0001 C CNN "LCSC"
@@
 $EndComp
 $Comp
-L Device:R_Small R?
+L Device:R_Small R13
 U 1 1 60DE8FF5
 P 9750 1250
-F 0 "R?" V 9554 1250 50  0000 C CNN
+F 0 "R13" V 9554 1250 50  0000 C CNN
 F 1 "22k" V 9645 1250 50  0000 C CNN
-F 2 "Resistor_SMD:R_0603_1608Metric_Pad0.98x0.95mm_HandSolder" H 9750 1250 50  0001 C CNN
+F 2 "Resistor_SMD:R_0603_1608Metric_Pad1.05x0.95mm_HandSolder" H 9750 1250 50  0001 C CNN
 F 3 "~" H 9750 1250 50  0001 C CNN
 F 4 "C31850" V 9750 1250 50  0001 C CNN "LCSC"
@@
 $EndComp
 $Comp
-L power:GND #PWR?
+L power:GND #PWR0140
 U 1 1 60DE9689
 P 9750 1350
-F 0 "#PWR?" H 9750 1100 50  0001 C CNN
+F 0 "#PWR0140" H 9750 1100 50  0001 C CNN
 F 1 "GND" H 9755 1177 50  0000 C CNN
 F 2 "" H 9750 1350 50  0001 C CNN
@@
 Vref=1.173\n(Vout=4.8V with 68k)\nVout=4.5V with 62k\nIout=23mA -> 1W,\n  -> 70°C over ambient
 $Comp
-L Device:R_Small R?
+L Device:R_Small R14
 U 1 1 60E7CBB2
 P 10050 950
-F 0 "R?" V 9854 950 50  0000 C CNN
+F 0 "R14" V 9854 950 50  0000 C CNN
 F 1 "DNP / 68k" V 9945 950 50  0000 C CNN
-F 2 "Resistor_SMD:R_0603_1608Metric_Pad0.98x0.95mm_HandSolder" H 10050 950 50  0001 C CNN
+F 2 "Resistor_SMD:R_0603_1608Metric_Pad1.05x0.95mm_HandSolder" H 10050 950 50  0001 C CNN
 F 3 "~" H 10050 950 50  0001 C CNN
 F 4 "C23231" V 10050 950 50  0001 C CNN "LCSC"
